Commit message: Rename links

File: urdf/robot.urdf (robot description, URDF)
Before this commit: robot diff_drive_robot, 5 links, 4 joints
Links:
- removed link castor_wheel
- removed link chassis
- removed link left_wheel
- removed link right_wheel
- added link castor_wheel_link; collision sphere radius=0.05; visual sphere radius=0.05
- added link chassis_link; collision box size=0.3 0.3 0.15; visual box size=0.3 0.3 0.15
- added link left_wheel_link; collision cylinder length=0.04 radius=0.05; visual cylinder length=0.04 radius=0.05
- added link right_wheel_link; collision cylinder length=0.04 radius=0.05; visual cylinder length=0.04 radius=0.05
Joints:
- joint castor_wheel_joint: child castor_wheel -> castor_wheel_link; parent chassis -> chassis_link
- joint chassis_joint: child chassis -> chassis_link
- joint left_wheel_joint: child left_wheel -> left_wheel_link
- joint right_wheel_joint: child right_wheel -> right_wheel_link
